File: 2025/03/ergogen/kb2/output/pcbs/pcb.kicad_pcb (KiCad board)
At the start: 2 copper layers, 235 x 72 mm, 54 parts

Commit message: more ergogen
Parts:
- added _2: , MountingHole_2.2mm_M2_Pad_Via, F.Cu at (109.0, 92.0)
- added _3: , MountingHole_2.2mm_M2_Pad_Via, F.Cu at (163.0, 92.0)
- added _4: , MountingHole_2.2mm_M2_Pad_Via, F.Cu at (232.0, 92.0)
- added _5: , MountingHole_2.2mm_M2_Pad_Via, F.Cu at (304.0, 92.0)
- added _6: , MountingHole_2.2mm_M2_Pad_Via, F.Cu at (163.0, 117.0)
- added _7: , MountingHole_2.2mm_M2_Pad_Via, F.Cu at (232.0, 117.0)
- added _8: , MountingHole_2.2mm_M2_Pad_Via, F.Cu at (197.5, 139.0)
- moved B1 3.00 mm to (197.5, 131.0)
Connections:
- D1 pad 1: GP0 -> GP10
- D10 pad 1: GP1 -> GP6
- D11 pad 1: GP0 -> GP10
- D12 pad 1: GP1 -> GP6
- D13 pad 1: GP0 -> GP10
- D14 pad 1: GP1 -> GP6
- D15 pad 1: GP0 -> GP10
- D16 pad 1: GP1 -> GP6
- D17 pad 1: GP0 -> GP10
- D18 pad 1: GP1 -> GP6
- D19 pad 1: GP0 -> GP10
- D2 pad 1: GP1 -> GP6
- D20 pad 1: GP1 -> GP6
- D21 pad 1: GP0 -> GP10
- D22 pad 1: GP1 -> GP6
- D23 pad 1: GP3 -> GP15
- D24 pad 1: GP3 -> GP15
- D25 pad 1: (no net) -> GP15
- D26 pad 1: (no net) -> GP15
- D3 pad 1: GP0 -> GP10
- D4 pad 1: GP1 -> GP6
- D5 pad 1: GP0 -> GP10
- D6 pad 1: GP1 -> GP6
- D7 pad 1: GP0 -> GP10
- D8 pad 1: GP1 -> GP6
- D9 pad 1: GP0 -> GP10
- S1 pad 1: GP4 -> GP1
- S10 pad 1: GP8 -> GP5
- S11 pad 1: GP8 -> GP5
- S12 pad 1: GP8 -> GP5
- S13 pad 1: GP7 -> GP4
- S14 pad 1: GP7 -> GP4
- S15 pad 1: GP6 -> GP3
- S16 pad 1: GP6 -> GP3
- S17 pad 1: GP5 -> GP2
- S18 pad 1: GP5 -> GP2
- S19 pad 1: GP4 -> GP1
- S2 pad 1: GP4 -> GP1
- S20 pad 1: GP4 -> GP1
- S21 pad 1: GP3 -> GP0
- S22 pad 1: GP3 -> GP0
- S23 pad 1: GP7 -> GP4
- S24 pad 1: GP8 -> GP5
- S25 pad 1: GP8 -> GP5
- S26 pad 1: GP7 -> GP4
- S3 pad 1: GP5 -> GP2
- S4 pad 1: GP5 -> GP2
- S5 pad 1: GP6 -> GP3
- S6 pad 1: GP6 -> GP3
- S7 pad 1: GP7 -> GP4
- S8 pad 1: GP7 -> GP4
- S9 pad 1: GP8 -> GP5

Commit message: change pins for keys
Parts:
- turned B1 to 180 degrees
Connections:
- D1 pad 1: GP10 -> GP9
- D10 pad 1: GP6 -> GP5
- D11 pad 1: GP10 -> GP22
- D12 pad 1: GP6 -> GP28
- D13 pad 1: GP10 -> GP22
- D14 pad 1: GP6 -> GP28
- D15 pad 1: GP10 -> GP22
- D16 pad 1: GP6 -> GP28
- D17 pad 1: GP10 -> GP22
- D18 pad 1: GP6 -> GP28
- D19 pad 1: GP10 -> GP22
- D2 pad 1: GP6 -> GP5
- D20 pad 1: GP6 -> GP28
- D21 pad 1: GP10 -> GP22
- D22 pad 1: GP6 -> GP28
- D3 pad 1: GP10 -> GP9
- D4 pad 1: GP6 -> GP5
- D5 pad 1: GP10 -> GP9
- D6 pad 1: GP6 -> GP5
- D7 pad 1: GP10 -> GP9
- D8 pad 1: GP6 -> GP5
- D9 pad 1: GP10 -> GP9
- S1 pad 1: GP1 -> GP10
- S10 pad 1: GP5 -> GP14
- S11 pad 1: GP5 -> GP16
- S12 pad 1: GP5 -> GP16
- S13 pad 1: GP4 -> GP17
- S14 pad 1: GP4 -> GP17
- S15 pad 1: GP3 -> GP18
- S16 pad 1: GP3 -> GP18
- S17 pad 1: GP2 -> GP19
- S18 pad 1: GP2 -> GP19
- S19 pad 1: GP1 -> GP20
- S2 pad 1: GP1 -> GP10
- S20 pad 1: GP1 -> GP20
- S21 pad 1: GP0 -> GP21
- S22 pad 1: GP0 -> GP21
- S23 pad 1: GP4 -> GP13
- S24 pad 1: GP5 -> GP14
- S25 pad 1: GP5 -> GP16
- S26 pad 1: GP4 -> GP17
- S3 pad 1: GP2 -> GP11
- S4 pad 1: GP2 -> GP11
- S5 pad 1: GP3 -> GP12
- S6 pad 1: GP3 -> GP12
- S7 pad 1: GP4 -> GP13
- S8 pad 1: GP4 -> GP13
- S9 pad 1: GP5 -> GP14

Commit message: finish wiring
Parts:
- moved _6 9.00 mm to (154.0, 117.0)
- moved _7 9.00 mm to (241.0, 117.0)
Connections:
- S1 pad 1: GP10 -> GP14
- S10 pad 1: GP14 -> GP10
- S11 pad 1: GP16 -> GP21
- S12 pad 1: GP16 -> GP21
- S13 pad 1: GP17 -> GP20
- S14 pad 1: GP17 -> GP20
- S15 pad 1: GP18 -> GP19
- S16 pad 1: GP18 -> GP19
- S17 pad 1: GP19 -> GP18
- S18 pad 1: GP19 -> GP18
- S19 pad 1: GP20 -> GP17
- S2 pad 1: GP10 -> GP14
- S20 pad 1: GP20 -> GP17
- S21 pad 1: GP21 -> GP16
- S22 pad 1: GP21 -> GP16
- S23 pad 1: GP13 -> GP11
- S24 pad 1: GP14 -> GP10
- S25 pad 1: GP16 -> GP21
- S26 pad 1: GP17 -> GP20
- S3 pad 1: GP11 -> GP13
- S4 pad 1: GP11 -> GP13
- S7 pad 1: GP13 -> GP11
- S8 pad 1: GP13 -> GP11
- S9 pad 1: GP14 -> GP10
