File: 2025/03/ergogen/kb2_v2/output/pcbs/pcb.kicad_pcb (KiCad board)
At the start: 2 copper layers, 235 x 72 mm, 61 parts

Commit message: ergogen ting
Parts:
- removed _8: , MountingHole_2.2mm_M2_Pad_Via
- added MCU1: , ProMicro, F.Cu at (197.5, 93.0)
- _1: value RPi_Pico_SMD_TH -> (none); footprint RPi_Pico_SMD_TH -> MountingHole_2.2mm_M2_Pad_Via
- moved _5 152.1 mm to (154.0, 117.0)
- moved _1 88.9 mm to (109.0, 92.0)
- moved _6 87.0 mm to (241.0, 117.0)
- moved _4 72.0 mm to (304.0, 92.0)
- moved _3 69.0 mm to (232.0, 92.0)
- moved _2 54.0 mm to (163.0, 92.0)
- moved _7 46.7 mm to (197.5, 134.0)
- moved B1 14.0 mm to (197.5, 117.0)
Connections:
- B1 pad 2: RUN -> RST
- _1 pad 1: GP0 -> (no net)

Commit message: init tvers
Parts:
- turned B1 to 0 degrees
Connections:
- net outer_bottom renamed outer_rbottom
- D1 pad 2: pinky_bottom -> pinky_lbottom
- D10 pad 2: inner_top -> inner_ltop
- D11 pad 2: inner_bottom -> inner_rbottom
- D12 pad 2: inner_top -> inner_rtop
- D13 pad 2: index_bottom -> index_rbottom
- D14 pad 2: index_top -> index_rtop
- D15 pad 2: middle_bottom -> middle_rbottom
- D16 pad 2: middle_top -> middle_rtop
- D17 pad 2: ring_bottom -> ring_rbottom
- D18 pad 2: ring_top -> ring_rtop
- D19 pad 2: pinky_bottom -> pinky_rbottom
- D2 pad 2: pinky_top -> pinky_ltop
- D20 pad 2: pinky_top -> pinky_rtop
- D22 pad 2: outer_top -> outer_rtop
- D23 pad 2: outer_top -> outer_lttop
- D24 pad 2: inner_top -> inner_lttop
- D25 pad 2: inner_top -> inner_rttop
- D26 pad 2: outer_top -> outer_rttop
- D3 pad 2: ring_bottom -> ring_lbottom
- D4 pad 2: ring_top -> ring_ltop
- D5 pad 2: middle_bottom -> middle_lbottom
- D6 pad 2: middle_top -> middle_ltop
- D7 pad 2: index_bottom -> index_lbottom
- D8 pad 2: index_top -> index_ltop
- D9 pad 2: inner_bottom -> inner_lbottom
- S1 pad 2: pinky_bottom -> pinky_lbottom
- S10 pad 2: inner_top -> inner_ltop
- S11 pad 2: inner_bottom -> inner_rbottom
- S12 pad 2: inner_top -> inner_rtop
- S13 pad 2: index_bottom -> index_rbottom
- S14 pad 2: index_top -> index_rtop
- S15 pad 2: middle_bottom -> middle_rbottom
- S16 pad 2: middle_top -> middle_rtop
- S17 pad 2: ring_bottom -> ring_rbottom
- S18 pad 2: ring_top -> ring_rtop
- S19 pad 2: pinky_bottom -> pinky_rbottom
- S2 pad 2: pinky_top -> pinky_ltop
- S20 pad 2: pinky_top -> pinky_rtop
- S22 pad 2: outer_top -> outer_rtop
- S23 pad 2: outer_top -> outer_lttop
- S24 pad 2: inner_top -> inner_lttop
- S25 pad 2: inner_top -> inner_rttop
- S26 pad 2: outer_top -> outer_rttop
- S3 pad 2: ring_bottom -> ring_lbottom
- S4 pad 2: ring_top -> ring_ltop
- S5 pad 2: middle_bottom -> middle_lbottom
- S6 pad 2: middle_top -> middle_ltop
- S7 pad 2: index_bottom -> index_lbottom
- S8 pad 2: index_top -> index_ltop
- S9 pad 2: inner_bottom -> inner_lbottom

Commit message: drag stuff
Parts:
- moved MCU1 2.50 mm to (197.5, 90.5)

Commit message: frood controller stuff
Parts:
- moved MCU1 1.50 mm to (197.5, 92.0)
Connections:
- net P0 renamed D0
- net P1 renamed D1
- net P10 renamed D10
- net P14 renamed D14
- net P15 renamed D15
- net P16 renamed D16
- net P18 renamed D18
- net P19 renamed D19
- net P2 renamed D2
- net P20 renamed D20
- net P21 renamed D21
- net P3 renamed D3
- net P4 renamed D4
- net P5 renamed D5
- net P6 renamed D6
- net P7 renamed D7
- net P8 renamed D8
- net P9 renamed D9

Commit message: route pcb
Connections:
- D1 pad 1: GP9 -> D23
- D10 pad 1: GP5 -> D29
- D11 pad 1: GP22 -> D9
- D12 pad 1: GP28 -> D2
- D13 pad 1: GP22 -> D9
- D14 pad 1: GP28 -> D2
- D15 pad 1: GP22 -> D9
- D16 pad 1: GP28 -> D2
- D17 pad 1: GP22 -> D9
- D18 pad 1: GP28 -> D2
- D19 pad 1: GP22 -> D9
- D2 pad 1: GP5 -> D29
- D20 pad 1: GP28 -> D2
- D21 pad 1: GP22 -> D9
- D22 pad 1: GP28 -> D2
- D23 pad 1: GP15 -> D21
- D24 pad 1: GP15 -> D21
- D25 pad 1: GP15 -> D21
- D26 pad 1: GP15 -> D21
- D3 pad 1: GP9 -> D23
- D4 pad 1: GP5 -> D29
- D5 pad 1: GP9 -> D23
- D6 pad 1: GP5 -> D29
- D7 pad 1: GP9 -> D23
- D8 pad 1: GP5 -> D29
- D9 pad 1: GP9 -> D23
- MCU1 pad 10: D14 -> D20
- MCU1 pad 11: D16 -> D23
- MCU1 pad 12: D10 -> D21
- MCU1 pad 13: D1 -> D12
- MCU1 pad 14: D0 -> D13
- MCU1 pad 15: GND -> D14
- MCU1 pad 16: GND -> D15
- MCU1 pad 17: D2 -> D16
- MCU1 pad 18: D3 -> Dp
- MCU1 pad 19: D4 -> D0
- MCU1 pad 20: D5 -> D1
- MCU1 pad 21: D6 -> GND
- MCU1 pad 22: D7 -> GND
- MCU1 pad 23: D8 -> D2
- MCU1 pad 24: D9 -> D3
- MCU1 pad 5: D21 -> D29
- MCU1 pad 6: D20 -> D28
- MCU1 pad 7: D19 -> D27
- MCU1 pad 8: D18 -> D26
- MCU1 pad 9: D15 -> D22
- S1 pad 1: GP14 -> D20
- S10 pad 1: GP10 -> D28
- S11 pad 1: GP21 -> D3
- S12 pad 1: GP21 -> D3
- S13 pad 1: GP20 -> D4
- S14 pad 1: GP20 -> D4
- S15 pad 1: GP19 -> D5
- S16 pad 1: GP19 -> D5
- S17 pad 1: GP18 -> D6
- S18 pad 1: GP18 -> D6
- S19 pad 1: GP17 -> D7
- S2 pad 1: GP14 -> D20
- S20 pad 1: GP17 -> D7
- S21 pad 1: GP16 -> D8
- S22 pad 1: GP16 -> D8
- S23 pad 1: GP11 -> D27
- S24 pad 1: GP10 -> D28
- S25 pad 1: GP21 -> D3
- S26 pad 1: GP20 -> D4
- S3 pad 1: GP13 -> D22
- S4 pad 1: GP13 -> D22
- S5 pad 1: GP12 -> D26
- S6 pad 1: GP12 -> D26
- S7 pad 1: GP11 -> D27
- S8 pad 1: GP11 -> D27
- S9 pad 1: GP10 -> D28
