File: 2025/03/ergogen/kb2_v2/pcbs/pcb.kicad_pcb (KiCad board)
At the start: 2 copper layers, 235 x 72 mm, 61 parts

Commit message: route pcb
Parts:
- removed _8: , MountingHole_2.2mm_M2_Pad_Via
- added MCU1: , ProMicro, F.Cu at (197.5, 92.0)
- _1: value RPi_Pico_SMD_TH -> (none); footprint RPi_Pico_SMD_TH -> MountingHole_2.2mm_M2_Pad_Via
- moved _5 152.1 mm to (154.0, 117.0)
- moved _1 88.9 mm to (109.0, 92.0)
- moved _6 87.0 mm to (241.0, 117.0)
- moved _4 72.0 mm to (304.0, 92.0)
- moved _3 69.0 mm to (232.0, 92.0)
- moved _2 54.0 mm to (163.0, 92.0)
- moved _7 46.7 mm to (197.5, 134.0)
- moved B1 14.0 mm to (197.5, 117.0), turned to 0 degrees
Connections:
- net outer_bottom renamed outer_rbottom
- B1 pad 2: RUN -> RST
- D1 pad 1: GP9 -> D23
- D1 pad 2: pinky_bottom -> pinky_lbottom
- D10 pad 1: GP5 -> D29
- D10 pad 2: inner_top -> inner_ltop
- D11 pad 1: GP22 -> D9
- D11 pad 2: inner_bottom -> inner_rbottom
- D12 pad 1: GP28 -> D2
- D12 pad 2: inner_top -> inner_rtop
- D13 pad 1: GP22 -> D9
- D13 pad 2: index_bottom -> index_rbottom
- D14 pad 1: GP28 -> D2
- D14 pad 2: index_top -> index_rtop
- D15 pad 1: GP22 -> D9
- D15 pad 2: middle_bottom -> middle_rbottom
- D16 pad 1: GP28 -> D2
- D16 pad 2: middle_top -> middle_rtop
- D17 pad 1: GP22 -> D9
- D17 pad 2: ring_bottom -> ring_rbottom
- D18 pad 1: GP28 -> D2
- D18 pad 2: ring_top -> ring_rtop
- D19 pad 1: GP22 -> D9
- D19 pad 2: pinky_bottom -> pinky_rbottom
- D2 pad 1: GP5 -> D29
- D2 pad 2: pinky_top -> pinky_ltop
- D20 pad 1: GP28 -> D2
- D20 pad 2: pinky_top -> pinky_rtop
- D21 pad 1: GP22 -> D9
- D22 pad 1: GP28 -> D2
- D22 pad 2: outer_top -> outer_rtop
- D23 pad 1: GP15 -> D21
- D23 pad 2: outer_top -> outer_lttop
- D24 pad 1: GP15 -> D21
- D24 pad 2: inner_top -> inner_lttop
- D25 pad 1: GP15 -> D21
- D25 pad 2: inner_top -> inner_rttop
- D26 pad 1: GP15 -> D21
- D26 pad 2: outer_top -> outer_rttop
- D3 pad 1: GP9 -> D23
- D3 pad 2: ring_bottom -> ring_lbottom
- D4 pad 1: GP5 -> D29
- D4 pad 2: ring_top -> ring_ltop
- D5 pad 1: GP9 -> D23
- D5 pad 2: middle_bottom -> middle_lbottom
- D6 pad 1: GP5 -> D29
- D6 pad 2: middle_top -> middle_ltop
- D7 pad 1: GP9 -> D23
- D7 pad 2: index_bottom -> index_lbottom
- D8 pad 1: GP5 -> D29
- D8 pad 2: index_top -> index_ltop
- D9 pad 1: GP9 -> D23
- D9 pad 2: inner_bottom -> inner_lbottom
- S1 pad 1: GP14 -> D20
- S1 pad 2: pinky_bottom -> pinky_lbottom
- S10 pad 1: GP10 -> D28
- S10 pad 2: inner_top -> inner_ltop
- S11 pad 1: GP21 -> D3
- S11 pad 2: inner_bottom -> inner_rbottom
- S12 pad 1: GP21 -> D3
- S12 pad 2: inner_top -> inner_rtop
- S13 pad 1: GP20 -> D4
- S13 pad 2: index_bottom -> index_rbottom
- S14 pad 1: GP20 -> D4
- S14 pad 2: index_top -> index_rtop
- S15 pad 1: GP19 -> D5
- S15 pad 2: middle_bottom -> middle_rbottom
- S16 pad 1: GP19 -> D5
- S16 pad 2: middle_top -> middle_rtop
- S17 pad 1: GP18 -> D6
- S17 pad 2: ring_bottom -> ring_rbottom
- S18 pad 1: GP18 -> D6
- S18 pad 2: ring_top -> ring_rtop
- S19 pad 1: GP17 -> D7
- S19 pad 2: pinky_bottom -> pinky_rbottom
- S2 pad 1: GP14 -> D20
- S2 pad 2: pinky_top -> pinky_ltop
- S20 pad 1: GP17 -> D7
- S20 pad 2: pinky_top -> pinky_rtop
- S21 pad 1: GP16 -> D8
- S22 pad 1: GP16 -> D8
- S22 pad 2: outer_top -> outer_rtop
- S23 pad 1: GP11 -> D27
- S23 pad 2: outer_top -> outer_lttop
- S24 pad 1: GP10 -> D28
- S24 pad 2: inner_top -> inner_lttop
- S25 pad 1: GP21 -> D3
- S25 pad 2: inner_top -> inner_rttop
- S26 pad 1: GP20 -> D4
- S26 pad 2: outer_top -> outer_rttop
- S3 pad 1: GP13 -> D22
- S3 pad 2: ring_bottom -> ring_lbottom
- S4 pad 1: GP13 -> D22
- S4 pad 2: ring_top -> ring_ltop
- S5 pad 1: GP12 -> D26
- S5 pad 2: middle_bottom -> middle_lbottom
- S6 pad 1: GP12 -> D26
- S6 pad 2: middle_top -> middle_ltop
- S7 pad 1: GP11 -> D27
- S7 pad 2: index_bottom -> index_lbottom
- S8 pad 1: GP11 -> D27
- S8 pad 2: index_top -> index_ltop
- S9 pad 1: GP10 -> D28
- S9 pad 2: inner_bottom -> inner_lbottom
- _1 pad 1: GP0 -> (no net)
Routing:
- net D8: track 0.00 -> 208.3 mm
- net D20: track 0.00 -> 206.6 mm
- net D7: track 0.00 -> 191.9 mm
- net D22: track 0.00 -> 190.4 mm
- net GP16: track 185.3 -> 0.00 mm
- net GP14: track 182.2 -> 0.00 mm
- net D6: track 0.00 -> 174.4 mm
- net D26: track 0.00 -> 173.4 mm
- net GP17: track 170.0 -> 0.00 mm
- net GP13: track 168.0 -> 0.00 mm
- net D27: track 0.00 -> 161.0 mm
- net D5: track 0.00 -> 157.9 mm
- net GP12: track 151.8 -> 0.00 mm
- net GP18: track 151.6 -> 0.00 mm
- net D4: track 0.00 -> 146.5 mm
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