File: 2025/03/ergogen/kb2_v4/pcbs/pcb.kicad_pcb (KiCad board)
At the start: 2 copper layers, 235 x 72 mm, 62 parts

Commit message: ergogen: add new column to v4 of keybaord
Parts:
- added D27: , ComboDiode, F.Cu at (241.0, 139.0)
- added D28: , ComboDiode, F.Cu at (259.0, 139.0)
- added S27: , PG1350, F.Cu at (241.0, 134.0)
- added S28: , PG1350, F.Cu at (259.0, 134.0)
- moved D23 180.2 mm to (331.0, 105.0)
- moved S23 180.2 mm to (331.0, 100.0)
- moved D24 167.0 mm to (331.0, 88.0)
- moved S24 167.0 mm to (331.0, 83.0)
- moved D25 51.0 mm to (172.0, 139.0)
- moved D26 51.0 mm to (190.0, 139.0)
- moved S25 51.0 mm to (172.0, 134.0)
- moved S26 51.0 mm to (190.0, 134.0)
- moved D11 33.0 mm to (190.0, 105.0)
- moved D12 33.0 mm to (190.0, 88.0)
- moved S11 33.0 mm to (190.0, 100.0)
- moved S12 33.0 mm to (190.0, 83.0)
- moved B1 18.0 mm to (215.5, 91.5)
- moved MCU1 18.0 mm to (215.5, 90.5)
- moved _2 18.0 mm to (181.0, 92.0)
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Connections:
- D1 pad 1: D23 -> D21
- D1 pad 2: pinky_lbottom -> outer_lbottom
- D10 pad 2: inner_ltop -> index_ltop
- D11 pad 1: D9 -> D21
- D11 pad 2: inner_rbottom -> inner_lbottom
- D12 pad 1: D2 -> D29
- D12 pad 2: inner_rtop -> inner_ltop
- D13 pad 2: index_rbottom -> inner_rbottom
- D14 pad 2: index_rtop -> inner_rtop
- D15 pad 2: middle_rbottom -> index_rbottom
- D16 pad 2: middle_rtop -> index_rtop
- D17 pad 2: ring_rbottom -> middle_rbottom
- D18 pad 2: ring_rtop -> middle_rtop
- D19 pad 2: pinky_rbottom -> ring_rbottom
- D2 pad 2: pinky_ltop -> outer_ltop
- D20 pad 2: pinky_rtop -> ring_rtop
- D21 pad 2: outer_rbottom -> pinky_rbottom
- D22 pad 2: outer_rtop -> pinky_rtop
- D23 pad 1: D21 -> D9
- D23 pad 2: outer_lttop -> outer_rbottom
- D24 pad 1: D21 -> D2
- D24 pad 2: inner_lttop -> outer_rtop
- D25 pad 1: D21 -> D1
- D25 pad 2: inner_rttop -> outer_lttop
- D26 pad 1: D21 -> D1
- D26 pad 2: outer_rttop -> inner_lttop
- D3 pad 1: D23 -> D21
- D3 pad 2: ring_lbottom -> pinky_lbottom
- D4 pad 2: ring_ltop -> pinky_ltop
- D5 pad 1: D23 -> D21
- D5 pad 2: middle_lbottom -> ring_lbottom
- D6 pad 2: middle_ltop -> ring_ltop
- D7 pad 1: D23 -> D21
- D7 pad 2: index_lbottom -> middle_lbottom
- D8 pad 2: index_ltop -> middle_ltop
- D9 pad 1: D23 -> D21
- D9 pad 2: inner_lbottom -> index_lbottom
- S1 pad 1: D20 -> D23
- S1 pad 2: pinky_lbottom -> outer_lbottom
- S10 pad 1: D28 -> D27
- S10 pad 2: inner_ltop -> index_ltop
- S11 pad 1: D3 -> D28
- S11 pad 2: inner_rbottom -> inner_lbottom
- S12 pad 1: D3 -> D28
- S12 pad 2: inner_rtop -> inner_ltop
- S13 pad 1: D4 -> D3
- S13 pad 2: index_rbottom -> inner_rbottom
- S14 pad 1: D4 -> D3
- S14 pad 2: index_rtop -> inner_rtop
- S15 pad 1: D5 -> D4
- S15 pad 2: middle_rbottom -> index_rbottom
- S16 pad 1: D5 -> D4
- S16 pad 2: middle_rtop -> index_rtop
- S17 pad 1: D6 -> D5
- S17 pad 2: ring_rbottom -> middle_rbottom
- S18 pad 1: D6 -> D5
- S18 pad 2: ring_rtop -> middle_rtop
- S19 pad 1: D7 -> D6
- S19 pad 2: pinky_rbottom -> ring_rbottom
- S2 pad 1: D20 -> D23
- S2 pad 2: pinky_ltop -> outer_ltop
- S20 pad 1: D7 -> D6
- S20 pad 2: pinky_rtop -> ring_rtop
- S21 pad 1: D8 -> D7
- S21 pad 2: outer_rbottom -> pinky_rbottom
- S22 pad 1: D8 -> D7
- S22 pad 2: outer_rtop -> pinky_rtop
- S23 pad 1: D27 -> D8
- S23 pad 2: outer_lttop -> outer_rbottom
- S24 pad 1: D28 -> D8
- S24 pad 2: inner_lttop -> outer_rtop
- S25 pad 1: D3 -> D27
- S25 pad 2: inner_rttop -> outer_lttop
- S26 pad 1: D4 -> D28
- S26 pad 2: outer_rttop -> inner_lttop
- S3 pad 1: D22 -> D20
- S3 pad 2: ring_lbottom -> pinky_lbottom
- S4 pad 1: D22 -> D20
- S4 pad 2: ring_ltop -> pinky_ltop
- S5 pad 1: D26 -> D22
- S5 pad 2: middle_lbottom -> ring_lbottom
- S6 pad 1: D26 -> D22
- S6 pad 2: middle_ltop -> ring_ltop
- S7 pad 1: D27 -> D26
- S7 pad 2: index_lbottom -> middle_lbottom
- S8 pad 1: D27 -> D26
- S8 pad 2: index_ltop -> middle_ltop
- S9 pad 1: D28 -> D27
- S9 pad 2: inner_lbottom -> index_lbottom
Routing:
- net D1: track 0.00 -> 169.4 mm
- net D23: track 121.9 -> 223.4 mm
- net D3: track 68.3 -> 132.8 mm
- net D29: track 121.3 -> 144.7 mm
- net GND: track 52.2 -> 32.4 mm
- net outer_ltop: track 0.00 -> 14.9 mm
- net outer_lbottom: track 0.00 -> 14.9 mm
- net D21: track 146.3 -> 144.2 mm
- net RST: track 21.3 -> 19.8 mm
- net D22: track 191.1 -> 190.4 mm
- net D6: track 175.0 -> 174.2 mm
- net D4: track 148.0 -> 148.8 mm
- net D8: track 209.4 -> 210.1 mm
Other:
- board size 235 x 72 mm -> 253 x 72 mm
