File: 2025/03/ergogen/kb2_v6-js/pcb/pcb.kicad_pcb (KiCad board)
At the start: 2 copper layers, 256 x 72 mm, 70 parts

Commit message: move screw holes to not interfere with switches
Parts:
- added _13: , Mount_Hole_2.2mm_Pad_Via, F.Cu at (217.0, 134.0)
- moved _6 148.0 mm to (181.0, 125.5)
- moved _7 90.0 mm to (325.0, 91.5)
- moved _11 57.1 mm to (235.0, 117.0)
- moved _10 25.5 mm to (235.0, 91.5)
- moved _4 24.4 mm to (199.0, 91.5)
- moved _3 23.8 mm to (181.0, 108.5)
- moved _2 18.0 mm to (181.0, 91.5)
- moved _12 10.2 mm to (253.0, 125.5)
- moved _8 6.82 mm to (253.0, 91.5)
- moved _9 1.97 mm to (253.0, 108.5)
Routing:
- net D1: track 172.4 -> 169.6 mm
- net D28: track 145.8 -> 148.0 mm
- net D27: track 162.7 -> 164.5 mm
- net D26: track 174.8 -> 176.4 mm
- net D6: track 177.4 -> 179.0 mm
- net D20: track 207.0 -> 208.5 mm
- net D5: track 161.3 -> 162.6 mm
- net D23: track 223.6 -> 224.8 mm
- net D22: track 191.3 -> 192.4 mm
- net D4: track 151.8 -> 150.8 mm
- net outer_lbottom: track 15.5 -> 14.9 mm
- net inner_lbottom: track 15.5 -> 14.9 mm
- net index_lbottom: track 15.5 -> 14.9 mm
- net ring_rtop: track 15.5 -> 14.9 mm
- net outer_rttop: track 15.5 -> 14.9 mm
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